File: v2315power/v2315power.kicad_pcb (KiCad board)
At the start: 2 copper layers, 82.5 x 50.8 mm, 12 parts, among them J1 Screw_Terminal_01x10, J2 Screw_Terminal_01x01, Q1 2N3904

Commit message: Update after testing
Connections:
- D2 pad 2: GNDREF -> Net-(D2-A)
- J1 pad 10: GNDREF -> Net-(D2-A)
Routing:
- net Net-(D2-A): track 0.00 -> 47.4 mm
- net GNDREF: track 47.4 -> 0.00 mm
Changed lines of the file:
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@@
   (net 6 "Net-(Q1-B)")
   (net 7 "Net-(J1-Pin_3)")
+  (net 8 "Net-(D2-A)")
   (footprint "TerminalBlock_Phoenix:TerminalBlock_Phoenix_MPT-0,5-10-2.54_1x10_P2.54mm_Horizontal" (layer "F.Cu")
     (at 92.12 80.99 -90)
@@
       (net 7 "Net-(J1-Pin_3)") (pinfunction "Pin_9") (pintype "passive"))
     (pad "10" thru_hole circle (at 22.86 0 270) (size 2.2 2.2) (drill 1.1) (layers "*.Cu" "*.Mask")
-      (net 4 "GNDREF") (pinfunction "Pin_10") (pintype "passive"))
+      (net 8 "Net-(D2-A)") (pinfunction "Pin_10") (pintype "passive"))
     (model "${KICAD6_3DMODEL_DIR}/TerminalBlock_Phoenix.3dshapes/TerminalBlock_Phoenix_MPT-0,5-10-2.54_1x10_P2.54mm_Horizontal.wrl"
       (offset (xyz 0 0 0))
@@
       (net 1 "Net-(D1-K)") (pinfunction "K") (pintype "passive"))
     (pad "2" thru_hole oval (at 15.24 0 180) (size 3.2 3.2) (drill 1.6) (layers "*.Cu" "*.Mask")
-      (net 4 "GNDREF") (pinfunction "A") (pintype "passive"))
+      (net 8 "Net-(D2-A)") (pinfunction "A") (pintype "passive"))
     (model "${KICAD6_3DMODEL_DIR}/Diode_THT.3dshapes/D_DO-201AD_P15.24mm_Horizontal.wrl"
       (offset (xyz 0 0 0))
@@
   )
   (segment (start 119.91 108.44) (end 119.69 108.66) (width 0.25) (layer "F.Cu") (net 1))
-  (segment (start 119.91 91.72) (end 119.91 108.44) (width 0.508) (layer "F.Cu") (net 1))
-  (segment (start 120.15 76.27) (end 120.15 91.48) (width 0.508) (layer "F.Cu") (net 1))
+  (segment (start 119.91 91.72) (end 119.91 108.44) (width 1.27) (layer "F.Cu") (net 1))
+  (segment (start 120.15 76.27) (end 120.15 91.48) (width 1.27) (layer "F.Cu") (net 1))
   (segment (start 120.15 91.48) (end 119.91 91.72) (width 0.25) (layer "F.Cu") (net 1))
-  (segment (start 92.12 80.99) (end 100.19 80.99) (width 0.508) (layer "F.Cu") (net 2))
+  (segment (start 92.12 80.99) (end 100.19 80.99) (width 1.27) (layer "F.Cu") (net 2))
   (segment (start 135.48 77.88) (end 135.36 77.76) (width 0.25) (layer "F.Cu") (net 2))
   (segment (start 132.82 77.76) (end 135.36 77.76) (width 0.25) (layer "F.Cu") (net 2))
   (segment (start 105.89 70.65) (end 125.71 70.65) (width 0.25) (layer "F.Cu") (net 2))
-  (segment (start 100.19 80.99) (end 104.91 76.27) (width 0.508) (layer "F.Cu") (net 2))
+  (segment (start 100.19 80.99) (end 104.91 76.27) (width 1.27) (layer "F.Cu") (net 2))
   (segment (start 125.71 70.65) (end 132.82 77.76) (width 0.25) (layer "F.Cu") (net 2))
   (segment (start 105.84 70.65) (end 105.89 70.65) (width 0.25) (layer "F.Cu") (net 2))
@@
   (segment (start 104.91 76.27) (end 104.91 71.63) (width 0.25) (layer "F.Cu") (net 2))
   (segment (start 104.91 71.63) (end 105.89 70.65) (width 0.25) (layer "F.Cu") (net 2))
-  (segment (start 98.92 96.23) (end 92.12 96.23) (width 0.508) (layer "F.Cu") (net 3))
-  (segment (start 104.45 101.76) (end 98.92 96.23) (width 0.508) (layer "F.Cu") (net 3))
-  (segment (start 104.45 108.66) (end 104.45 101.76) (width 0.508) (layer "F.Cu") (net 3))
-  (segment (start 104.67 91.72) (end 112.14 99.19) (width 0.508) (layer "F.Cu") (net 4))
-  (segment (start 101.49 113.22) (end 92.12 103.85) (width 0.508) (layer "F.Cu") (net 4))
-  (segment (start 112.14 99.19) (end 112.14 111.4) (width 0.508) (layer "F.Cu") (net 4))
-  (segment (start 110.32 113.22) (end 101.49 113.22) (width 0.508) (layer "F.Cu") (net 4))
-  (segment (start 112.14 111.4) (end 110.32 113.22) (width 0.508) (layer "F.Cu") (net 4))
+  (segment (start 98.92 96.23) (end 92.12 96.23) (width 1.27) (layer "F.Cu") (net 3))
+  (segment (start 104.45 101.76) (end 98.92 96.23) (width 1.27) (layer "F.Cu") (net 3))
+  (segment (start 104.45 108.66) (end 104.45 101.76) (width 1.27) (layer "F.Cu") (net 3))
   (segment (start 151.39 93.33) (end 151.39 100.93) (width 0.25) (layer "F.Cu") (net 5))
   (segment (start 151.39 100.93) (end 145.62 106.7) (width 0.25) (layer "F.Cu") (net 5))
@@
   (segment (start 150.12 80.65) (end 152.89 77.88) (width 0.25) (layer "F.Cu") (net 6))
   (segment (start 150.12 93.33) (end 150.12 80.65) (width 0.25) (layer "F.Cu") (net 6))
-  (segment (start 88.48 91.15) (end 86.18 88.85) (width 0.508) (layer "F.Cu") (net 7))
-  (segment (start 86.18 99.55) (end 87.94 101.31) (width 0.508) (layer "F.Cu") (net 7))
-  (segment (start 86.18 88.85) (end 86.18 99.55) (width 0.508) (layer "F.Cu") (net 7))
-  (segment (start 92.12 86.07) (end 88.2 86.07) (width 0.508) (layer "F.Cu") (net 7))
+  (segment (start 86.18 99.55) (end 87.94 101.31) (width 1.27) (layer "F.Cu") (net 7))
+  (segment (start 86.18 88.09) (end 86.18 99.55) (width 1.27) (layer "F.Cu") (net 7))
+  (segment (start 92.12 86.07) (end 88.2 86.07) (width 1.27) (layer "F.Cu") (net 7))
   (segment (start 92.69 91.72) (end 92.12 91.15) (width 0.25) (layer "F.Cu") (net 7))
-  (segment (start 86.18 88.09) (end 86.18 88.85) (width 0.508) (layer "F.Cu") (net 7))
-  (segment (start 92.12 91.15) (end 88.48 91.15) (width 0.25) (layer "F.Cu") (net 7))
-  (segment (start 88.2 86.07) (end 86.18 88.09) (width 0.508) (layer "F.Cu") (net 7))
-  (segment (start 87.94 101.31) (end 92.12 101.31) (width 0.508) (layer "F.Cu") (net 7))
+  (segment (start 88.48 91.15) (end 92.12 91.15) (width 1.27) (layer "F.Cu") (net 7))
+  (segment (start 86.18 88.85) (end 88.48 91.15) (width 1.27) (layer "F.Cu") (net 7))
+  (segment (start 88.2 86.07) (end 86.18 88.09) (width 1.27) (layer "F.Cu") (net 7))
+  (segment (start 87.94 101.31) (end 92.12 101.31) (width 1.27) (layer "F.Cu") (net 7))
+  (segment (start 104.67 91.72) (end 112.14 99.19) (width 1.27) (layer "F.Cu") (net 8))
+  (segment (start 101.49 113.22) (end 92.12 103.85) (width 1.27) (layer "F.Cu") (net 8))
+  (segment (start 112.14 99.19) (end 112.14 111.4) (width 1.27) (layer "F.Cu") (net 8))
+  (segment (start 110.32 113.22) (end 101.49 113.22) (width 1.27) (layer "F.Cu") (net 8))
+  (segment (start 112.14 111.4) (end 110.32 113.22) (width 1.27) (layer "F.Cu") (net 8))
   (zone (net 4) (net_name "GNDREF") (layer "B.Cu") (hatch edge 0.5)
     (connect_pads (clearance 0.5))
