File: 2310interface/2310interface.kicad_pcb (KiCad board)
At the start: 2 copper layers, 179.8 x 99.3 mm, 63 parts, among them J4 Screw_Terminal_01x04, Q1 Q_NMOS_DSG, Q2 2N3904, SW1 SW_SPDT, U1 LD1117S50TR_SOT223

Commit message: Update after testing
Other:
- board text added: "100nF"
- board text added: "10K"
- board text added: "10uF"
- board text added: "2.7K"
- board text added: "2N3904"
- board text added: "47K"
- board text added: "LD1117S50"
- board text added: "Q1"
Changed lines of the file:
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@@
     (property "ki_keywords" "R res resistor")
     (attr smd)
-    (fp_text reference "R5" (at 0 -1.65 90) (layer "F.SilkS")
+    (fp_text reference "R5" (at -0.0625 3.13 90) (layer "F.SilkS")
         (effects (font (size 1 1) (thickness 0.15)))
     )
@@
     (property "ki_keywords" "REGULATOR LDO 5.0V")
     (attr smd)
-    (fp_text reference "U1" (at 0 -4.5) (layer "F.SilkS")
+    (fp_text reference "U1" (at -0.26 4.25) (layer "F.SilkS")
         (effects (font (size 1 1) (thickness 0.15)))
     )
@@
     (property "ki_keywords" "cap capacitor")
     (attr smd)
-    (fp_text reference "C2" (at 0 -1.68 90) (layer "F.SilkS")
+    (fp_text reference "C2" (at 3.5 0 -180) (layer "F.SilkS")
         (effects (font (size 1 1) (thickness 0.15)))
     )
@@
     (property "ki_keywords" "R res resistor")
     (attr smd)
-    (fp_text reference "R7" (at 0 -1.65) (layer "F.SilkS")
+    (fp_text reference "R7" (at -0.17 -3.09) (layer "F.SilkS")
         (effects (font (size 1 1) (thickness 0.15)))
     )
@@
     (property "ki_keywords" "R res resistor")
     (attr smd)
-    (fp_text reference "R1" (at 0 -1.65 90) (layer "F.SilkS")
+    (fp_text reference "R1" (at 0.08 -3.34 90) (layer "F.SilkS")
         (effects (font (size 1 1) (thickness 0.15)))
     )
@@
     (property "ki_keywords" "R res resistor")
     (attr smd)
-    (fp_text reference "R6" (at 0 -1.65 90) (layer "F.SilkS")
+    (fp_text reference "R6" (at 0.03 -1.64 90) (layer "F.SilkS")
         (effects (font (size 1 1) (thickness 0.15)))
     )
@@
     (property "ki_keywords" "R res resistor")
     (attr smd)
-    (fp_text reference "R4" (at 0 -1.65 90) (layer "F.SilkS")
+    (fp_text reference "R4" (at 0.04 3.21 90) (layer "F.SilkS")
         (effects (font (size 1 1) (thickness 0.15)))
     )
@@
     (effects (font (size 1.5 1.5) (thickness 0.3) bold) (justify left bottom))
   )
+  (gr_text "LD1117S50" (at 126.46 119.86) (layer "F.SilkS")
+    (effects (font (size 1 1) (thickness 0.15)) (justify left bottom))
+  )
+  (gr_text "10K" (at 131.57 100.76 -90) (layer "F.SilkS")
+    (effects (font (size 1 1) (thickness 0.15)) (justify left bottom))
+  )
+  (gr_text "100nF" (at 136.19 111.84) (layer "F.SilkS")
+    (effects (font (size 1 1) (thickness 0.15)) (justify left bottom))
+  )
   (gr_text "Cable to 2310" (at 97.2 49.59) (layer "F.SilkS")
     (effects (font (face "Arial") (size 2.54 2.54) (thickness 0.3) bold) (justify left bottom))
@@
     (effects (font (size 1 1) (thickness 0.15)) (justify left bottom))
   )
+  (gr_text "47K" (at 147.15 102.85 90) (layer "F.SilkS")
+    (effects (font (size 1 1) (thickness 0.15)) (justify left bottom))
+  )
   (gr_text "Virtual 2315 Cartridge Facility" (at 77.15 68.27) (layer "F.SilkS")
     (effects (font (face "Arial") (size 3.81 3.81) (thickness 0.3) bold) (justify left bottom))
@@
     (effects (font (size 1 1) (thickness 0.15)) (justify left bottom))
   )
+  (gr_text "2.7K" (at 139.04 96.03) (layer "F.SilkS")
+    (effects (font (size 1 1) (thickness 0.15)) (justify left bottom))
+  )
+  (gr_text "2N3904" (at 136.88 106.05) (layer "F.SilkS")
+    (effects (font (size 1 1) (thickness 0.15)) (justify left bottom))
+  )
+  (gr_text "10K" (at 152.29 93.16 90) (layer "F.SilkS")
+    (effects (font (size 1 1) (thickness 0.15)) (justify left bottom))
+  )
   (gr_text "-Lamp" (at 156.87 111.19 90) (layer "F.SilkS")
     (effects (font (size 1.5 1.5) (thickness 0.3) bold) (justify left bottom))
   )
+  (gr_text "Q1" (at 162.51 100.4) (layer "F.SilkS")
+    (effects (font (size 1 1) (thickness 0.15)) (justify left bottom))
+  )
+  (gr_text "2.7K" (at 147.03 97.75 90) (layer "F.SilkS")
+    (effects (font (size 1 1) (thickness 0.15)) (justify left bottom))
+  )
+  (gr_text "10uF" (at 136.43 120.44) (layer "F.SilkS")
+    (effects (font (size 1 1) (thickness 0.15)) (justify left bottom))
+  )
   (gr_text "Ground" (at 162.16 110.03 90) (layer "F.SilkS")

Commit message: Fix defect in board
Inadvertent connection of +12V to the Unlock lamp driver
also increased current capacity for Unlock lamp traces
Parts:
- C1: value C -> 100nF
- C2: value C -> 10uF
- K1: renamed from REF**; value Relay_SPDT_Finder_36.11 -> Relay_SPDT
- renumbered B10 to AB10, B12 to AB12, B13 to AB13, B02 to AB2, B03 to AB3, B04 to AB4, B05 to AB5, B07 to AB7, B08 to AB8, B09 to AB9, D10 to AD10, D11 to AD11, D12 to AD12, D13 to AD13, D02 to AD2, D04 to AD4, D05 to AD5, D06 to AD6, D07 to AD7, D09 to AD9
Connections:
- net Ref12 renamed Net-(Q1-D)
- AD7 pad 1: unconnected-(D7a1-Pin_1-Pad1) -> GND
- ConnB1 pad 39: Net-(J4-Pin_1) -> Net-(ConnB1-Pin_39)
- D7 pad 1: GND -> unconnected-(D7-Pin_1-Pad1)
- Q1 pad 3: Net-(J4-Pin_1) -> Net-(ConnB1-Pin_39)
- R1 pad 1: Net-(J4-Pin_1) -> Net-(ConnB1-Pin_39)
Routing:
- net Net-(J4-Pin_1): track 246.2 -> 20.6 mm, vias 2 -> 0
- net Net-(ConnB1-Pin_39): track 0.00 -> 153.8 mm, vias 0 -> 8
- net Net-(ConnA1-Pin_36): track 138.1 -> 156.9 mm, vias 1 -> 4
- net Net-(AD2-Pin_1): track 125.4 -> 136.2 mm
- net GND: track 124.9 -> 120.2 mm
- net Net-(B13-Pin_1): track 143.4 -> 140.3 mm
- net Net-(Q1-D): track 35.6 -> 35.4 mm, vias 2 -> 1
Other:
- board text added: "B02"
- board text added: "B03"
- board text added: "B04"
- board text added: "B05"
- board text added: "B07"
- board text added: "B08"
- board text added: "B09"
- board text added: "B10"
- board text added: "B12"
- board text added: "B13"
- board text added: "B13 B12 B11 B10 B09 B08 B07 B06 B05 B04 B03 B02"
- board text added: "D02"
- board text added: "D04"
- board text added: "D05"
- board text added: "D06"
- board text added: "D07"
- board text added: "D09"
- board text added: "D10"
- board text added: "D11"
- board text added: "D12"
- board text added: "D13"
- board text added: "D13 D12 D11 D10 D09 D08 D07 D06 D05 D04 D03 D02"
