File: 2310interface/2310interface.kicad_pcb (KiCad board)
At the start: 2 copper layers, 179.8 x 99.3 mm, 63 parts, among them J4 Screw_Terminal_01x04, K1 Relay_SPDT, Q1 Q_NMOS_DSG, Q2 2N3904, SW1 SW_SPDT, U1 LD1117S50TR_SOT223

Commit message: Version with electronic switch
bidirectional analog electronic switch to connect disk and 1130 signals together when in real disk mode to eliminate delays and other issues for signals that simply pass through. These can still be observed inside the FPGA which is important for shadowing the disk rotation and arm movement of the disk.
Parts:
- added C3: .1uF, Capacitor_SMD:C_0805_2012Metric, B.Cu at (94.2, 76.5)
- added C4: .1uF, Capacitor_SMD:C_0805_2012Metric, B.Cu at (55.9, 34.7)
- added U2: TMUX1112PWR, footprints:PW0016A-MFG, F.Cu at (94.2, 76.3)
- added U3: TMUX1112PWR, footprints:PW0016A-MFG, F.Cu at (56.0, 34.5)
Routing:
- net Net-(ConnA1-Pin_18): track 110.2 -> 248.0 mm, vias 4 -> 8
- net Net-(SW1-A): track 53.9 -> 185.0 mm, vias 4 -> 12
- net Net-(B2-Pin_1): track 87.4 -> 203.6 mm, vias 0 -> 5
- net Net-(AB12-Pin_1): track 46.5 -> 144.5 mm
- net Net-(B12-Pin_1): track 79.4 -> 159.5 mm, vias 0 -> 2
- net Net-(AB10-Pin_1): track 79.2 -> 152.3 mm, vias 2 -> 5
- net Net-(AD6-Pin_1): track 101.0 -> 170.9 mm, vias 0 -> 2
- net Net-(AB4-Pin_1): track 49.3 -> 117.6 mm, vias 2 -> 7
- net Net-(B4-Pin_1): track 113.2 -> 167.9 mm, vias 0 -> 2
- net Net-(AB7-Pin_1): track 89.7 -> 139.4 mm, vias 1 -> 4
- net Net-(ConnB1-Pin_25): track 63.9 -> 110.0 mm, vias 0 -> 1
- net Net-(B10-Pin_1): track 125.0 -> 168.1 mm, vias 2 -> 4
- net Net-(B7-Pin_1): track 117.9 -> 160.3 mm, vias 2 -> 4
- net GND: track 120.2 -> 156.5 mm, vias 31 -> 41
- net Net-(AD4-Pin_1): track 55.6 -> 89.6 mm, vias 2 -> 4
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