File: 2310interface/2310interface.kicad_sch (KiCad schematic)
At the start: 63 parts, among them J4 Screw_Terminal_01x04, K1 Relay_SPDT, Q1 Q_NMOS_DSG, Q2 2N3904, SW1 SW_SPDT, U1 LD1117S50TR_SOT223

Commit message: Version with electronic switch
bidirectional analog electronic switch to connect disk and 1130 signals together when in real disk mode to eliminate delays and other issues for signals that simply pass through. These can still be observed inside the FPGA which is important for shadowing the disk rotation and arm movement of the disk.
Parts:
- added C3, C4: .1uF, Capacitor_SMD:C_0805_2012Metric, symbol Device:C_Small
- added U2, U3: TMUX1112PWR, footprints:PW0016A-MFG, symbol 2026-07-28_13-09-32:TMUX1112PWR
Connections:
- net GND: now also C3.2, C4.2, U2.5 (GND), U3.10 (D3), U3.11 (S3), U3.5 (GND)
- net at C2.1, R6.1, SW1.1 (A)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: now also C3.1, C4.1, U2.13 (VDD), U3.13 (VDD)
- net at AD4.1 (Pin_1), ConnB1.29 (Pin_29): now also U2.2 (D1)
- net at ConnA1.18 (Pin_18), K1.A1, SW1.2 (B): now also U2.1 (SEL1), U2.16 (SEL2), U2.8 (SEL4), U2.9 (SEL3), U3.1 (SEL1), U3.16 (SEL2), U3.8 (SEL4), U3.9 (SEL3)
- net at B2.1 (Pin_1), ConnA1.34 (Pin_34): now also U3.7 (D4)
- net at AB4.1 (Pin_1), ConnB1.27 (Pin_27): now also U2.10 (D3)
- net at B4.1 (Pin_1), ConnA1.40 (Pin_40): now also U2.11 (S3)
- net at AB12.1 (Pin_1), ConnA1.12 (Pin_12): now also U3.14 (S2)
- net at B7.1 (Pin_1), ConnA1.14 (Pin_14): now also U2.15 (D2)
- net at AB7.1 (Pin_1), ConnA1.22 (Pin_22): now also U2.14 (S2)
- net at AB2.1 (Pin_1), ConnA1.26 (Pin_26): now also U3.6 (S4)
- net at B10.1 (Pin_1), ConnA1.28 (Pin_28): now also U2.6 (S4)
- net at AB10.1 (Pin_1), ConnA1.32 (Pin_32): now also U2.7 (D4)
- net at AD6.1 (Pin_1), ConnA1.8 (Pin_8): now also U3.3 (S1)
- net at B12.1 (Pin_1), ConnB1.19 (Pin_19): now also U3.15 (D2)
- net at ConnB1.25 (Pin_25), D6.1 (Pin_1): now also U3.2 (D1)
- net at ConnB1.5 (Pin_5), D4.1 (Pin_1): now also U2.3 (S1)
- no-connect marks 0 -> 54
Other:
- note added: "Access Go Access Read Rev/Fwd step 10/20 step"
- note added: "Sector Index N/C Home"
